File: pcb/board/board.kicad_sch (KiCad schematic)
At the start: 117 parts, among them J1 (A) USB_C_Receptacle_USB2.0_1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, J10 OLED_128x32, J11 LCD_128x160, J12 Conn_01x03, J13 AudioJack3, J14 Micro_SD_Card, J2 (B) USB_C_Receptacle_USB2.0_1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, J3 (C) USB_C_Receptacle_USB2.0_1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, J4 Conn_01x03, J5 Conn_01x03, J6 Conn_01x20, J7 Conn_01x20, J8 Conn_01x20, J9 Conn_01x20, SW1 SW_Push, SW2 SW_Push, SW3 Switch, SW4 Switch, SW5 Switch, SW6 RotaryEncoder_Switch, U1 RP2040, U2 NCP1117-3.3_SOT223, U3 W25Q128JVS, U4 NCP1117-3.3_SOT223, U5 RP2040, U6 W25Q128JVS, U7 PCM5101A, U8 TLV70033_SOT23-5, Y1 12MHz, Y2 12MHz

Commit message: reassign pins and mcu spi connection (and uart backup!)!
Parts:
- added J15: Conn_02x06_Row_Letter_Last, symbol Connector_Generic:Conn_02x06_Row_Letter_Last
- added J16: Conn_02x04_Row_Letter_Last, symbol Connector_Generic:Conn_02x04_Row_Letter_Last
Connections:
- net GPIO0_A: now also J15.1a (Pin_1a), J15.5a (Pin_5a); no longer J12.1 (Pin_1)
- net GPIO0_B: now also J15.4b (Pin_4b), J15.5b (Pin_5b); no longer J11.6 (DC)
- net GPIO10_A: now also J12.1 (Pin_1); no longer J14.5 (CLK), R21.1
- net GPIO10_B: now also J11.3 (SCL)
- net GPIO11_B: now also J11.4 (SDA)
- net GPIO12_A: now also J14.7 (DAT0); no longer J10.4 (SDA)
- net GPIO12_B: now also J11.5 (RST)
- net GPIO13_A: now also J14.2 (DAT3/CD); no longer J10.3 (SCL)
- net GPIO13_B: now also J11.8 (BLK)
- net GPIO14_A: now also J14.5 (CLK), R21.1
- net GPIO16_A: now also J16.1a (Pin_1a), J16.3a (Pin_3a)
- net GPIO16_B: now also J16.2b (Pin_2b), J16.3b (Pin_3b)
- net GPIO17_A: now also J16.2a (Pin_2a), J16.4a (Pin_4a)
- net GPIO17_B: now also J16.1b (Pin_1b), J16.4b (Pin_4b)
- net GPIO18_A: now also J10.4 (SDA)
- net GPIO19_A: now also J10.3 (SCL)
- net GPIO1_A: now also J15.2a (Pin_2a); no longer SW3.1
- net GPIO1_B: now also J15.2b (Pin_2b); no longer J11.7 (CS)
- net GPIO2_A: now also J15.3a (Pin_3a); no longer SW4.1
- net GPIO2_B: now also J15.3b (Pin_3b); no longer J11.3 (SCL)
- net GPIO3_A: now also J15.4a (Pin_4a), J15.6a (Pin_6a); no longer SW5.1
- net GPIO3_B: now also J15.1b (Pin_1b), J15.6b (Pin_6b); no longer J11.4 (SDA)
- net GPIO4_A: now also SW3.1; no longer SW6.S1
- net GPIO4_B: no longer J11.5 (RST)
- net GPIO5_A: now also SW4.1; no longer SW6.A
- net GPIO5_B: no longer J11.8 (BLK)
- net GPIO6_A: now also SW5.1; no longer SW6.B
- net GPIO7_A: now also SW6.S1
- net GPIO8_A: now also SW6.A; no longer J14.7 (DAT0)
- net GPIO8_B: now also J11.6 (DC)
- net GPIO9_A: now also SW6.B; no longer J14.2 (DAT3/CD)
- net GPIO9_B: now also J11.7 (CS)
Other:
- note added: "0-3: SPI0 MCU (to implement) 8-13: LCD 128x160 Display 16-17: UART0 MCU (backup) (to implement) 23-25: RGB, Board, Boot LEDS"
- note added: "0-3: SPI0 MCU 4-10: Buttons 11-14: Micro SD Card 18-19: OLED 128x32 Display 16-17: UART0 MCU (backup) 23-25: RGB, Board, Boot LEDS 26-28: Audio"
- note added: "GPIO13: BLK, generic GPIO9: CS, SPI1 CSn GPIO8: DC, generic GPIO12: RST, generic GPIO11: SDA, SPI1 TX (MOSI) GPIO10: SCL, SPI1 SCK"
- note added: "GPIO18: I2C0 SDA GPIO19: I2C0 SCL"
- note added: "SPI Interface DAT0-RX-MISO (12) CMD-TX-MOSI (11) DAT3-CS (13) CLK-SCK (14)"
- note removed: "0-5: LCD 128x160 Display 23: RGB LEDS 24: Board LED 25: Boot LED"
- note removed: "0-6: Buttons 8-11: Micro SD Card 12-13: OLED 128x32 Display 23: RGB LEDS 24: Board LED 25: Boot LED 26-28: Audio"
- note removed: "GPIO12: I2C0 SDA GPIO13: I2C0 SCL"
- note removed: "GPIO5: BLK, generic GPIO1: CS, SPI0 CSn GPIO0: DC, generic GPIO4: RST, generic GPIO3: SDA, SPI0 TX (MOSI) GPIO2: SCL, SPI0 SCK"
- note removed: "SPI Interface DAT0-RX-MISO (8) CMD-TX-MOSI (11) DAT3-CS (9) CLK-SCK(10)"
- company: (none) -> HenryLi-0
- title: (none) -> River Board

Commit message: 08052026 - reassign pins and more audio stuff!
Parts:
- removed C45: 2.2uF, Capacitor_SMD:C_0402_1005Metric, symbol Device:C
- removed D5, D6, D7, D8: Diode, Diode_THT:D_DO-35_SOD27_P7.62mm_Horizontal, symbol ScottoKeebs:Placeholder_Diode
- removed J12: Conn_01x03, Connector_PinHeader_2.54mm:PinHeader_1x03_P2.54mm_Vertical, symbol Connector_Generic:Conn_01x03
- removed J15: Conn_02x06_Row_Letter_Last, symbol Connector_Generic:Conn_02x06_Row_Letter_Last
- removed J16: Conn_02x04_Row_Letter_Last, symbol Connector_Generic:Conn_02x04_Row_Letter_Last
- added C50, C51, C52, C53, C54, C55: 1uF, Capacitor_SMD:C_0402_1005Metric, symbol Device:C
- added D5: LED, symbol Device:LED
- added J12: AudioJack2, symbol Connector_Audio:AudioJack2
- added R24: 330, Resistor_SMD:R_0402_1005Metric, symbol Device:R
- added U9: TPA6132A2RTE, Package_DFN_QFN:WQFN-16-1EP_3x3mm_P0.5mm_EP1.6x1.6mm_ThermalVias, symbol Amplifier_Audio:TPA6132A2RTE
Connections:
- net GPIO17_A is gone; now on net GPIO16_B: J7.19 (Pin_19), U1.28 (GPIO17)
- net GPIO17_B is gone; now on net GPIO16_A: J9.19 (Pin_19), U5.28 (GPIO17)
- net GPIO1_B is gone; now on net GPIO1_A: J8.2 (Pin_2), U5.3 (GPIO1)
- net GPIO2_B is gone; now on net GPIO2_A: J8.4 (Pin_4), U5.4 (GPIO2)
- net GPIO3_A is gone; now on net GPIO0_B: J6.5 (Pin_5), U1.5 (GPIO3)
- net GPIO3_B is gone; now on net GPIO0_A: J8.5 (Pin_5), U5.5 (GPIO3)
- net +3V3_AUDIO: now also U9.14 (VDD)
- net GND: now also SW3.2, SW4.2, SW5.2, SW6.S2, C51.1, C54.1, C55.1, R24.2, U9.10 (PGND), U9.17 (EP); no longer J13.S
- net GPIO10_A: now also D5.2 (A)
- net GPIO21_A: now also U9.6 (G0)
- net GPIO22_A: now also U9.7 (G1)
- net GPIO29_C3_A: now also U9.13 (EN)
- net at R19.2: now also C52.1; no longer J13.T
- new net: C50.1, U9.11 (CPP)
- new net: C50.2, U9.9 (CPN)
- new net: C53.1, R20.2
- new net: C55.2, U9.2 (INL+)
- new net: C51.2, U9.8 (HPVSS)
- new net: J13.R, U9.5 (OUTR)
- new net: J12.T, J13.T, U9.16 (OUTL)
- new net: C52.2, U9.1 (INL-)
- new net: C53.2, U9.4 (INR-)
- new net: C44.1, U9.12 (HPVDD)
- new net: C54.2, U9.3 (INR+)
- new net: D5.1 (K), R24.1
- new net SGND: J12.S, J13.S, U9.15 (SGND)
Other:
- note added: "0-3: SPI0 MCU 4-10: Buttons 11-14: Micro SD Card 16-17: UART0 MCU (backup) 18-19: OLED 128x32 Display 23-25: RGB, Board, Boot LEDS 21-22, 26-29: Audio"
- note added: "0-3: SPI0 MCU 8-13: LCD 128x160 Display 16-17: UART0 MCU (backup) 23-25: RGB, Board, Boot LEDS"
- note added: "TODO: DOUBLE CHECK AMP POWER!!!"
- note removed: "0-3: SPI0 MCU (to implement) 8-13: LCD 128x160 Display 16-17: UART0 MCU (backup) (to implement) 23-25: RGB, Board, Boot LEDS"
- note removed: "0-3: SPI0 MCU 4-10: Buttons 11-14: Micro SD Card 18-19: OLED 128x32 Display 16-17: UART0 MCU (backup) 23-25: RGB, Board, Boot LEDS 26-28: Audio"
- moved on the sheet: C35, C36, C37, C38, C39, C40, C41, C42, C43, C48, J10, J11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
