File: pcb/board/board.kicad_sch (KiCad schematic)
At the start: 121 parts, among them J1 (A) USB_C_Receptacle_USB2.0_1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, J10 OLED_128x32, J11 LCD_128x160, J12 AudioJack2, J13 AudioJack3, J14 Micro_SD_Card, J2 (B) USB_C_Receptacle_USB2.0_1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, J3 (C) USB_C_Receptacle_USB2.0_1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, J4 Conn_01x03, J5 Conn_01x03, J6 Conn_01x20, J7 Conn_01x20, J8 Conn_01x20, J9 Conn_01x20, SW1 SW_Push, SW2 SW_Push, SW3 Switch, SW4 Switch, SW5 Switch, SW6 RotaryEncoder_Switch, U1 RP2040, U2 NCP1117-3.3_SOT223, U3 W25Q128JVS, U4 NCP1117-3.3_SOT223, U5 RP2040, U6 W25Q128JVS, U7 PCM5101A, U8 TLV70033_SOT23-5, U9 TPA6132A2RTE, Y1 12MHz, Y2 12MHz

Commit message: footprint assigning and wrapping up schematic work!
Parts:
- removed C52, C53, C54, C55: 1uF, Capacitor_SMD:C_0402_1005Metric, symbol Device:C
- removed D1, D2: D_Schottky, symbol Device:D_Schottky
- removed J12: AudioJack2, symbol Connector_Audio:AudioJack2
- added C45, C49: 1uF, Capacitor_SMD:C_0603_1608Metric, symbol Device:C
- added D1, D2: SS14, Diode_SMD:D_SMA, symbol Diode:SS14
- added R25, R26: 330, Resistor_SMD:R_0402_1005Metric, symbol Device:R
- C1, C10, C11, C12, C13, C14, C17, C18, C19, C2, C20, C23, C24, C25, C26, C27, C28, C29, C3, C30, C31, C32, C33, C34, C35, C36, C37, C38, C39, C4, C40, C41, C42, C43, C44, C46, C47, C48, C5, C50, C51, C6, C7, C8, C9: footprint Capacitor_SMD:C_0402_1005Metric -> Capacitor_SMD:C_0603_1608Metric
- C15, C16, C21, C22: value 15uF -> 33pF; footprint Capacitor_SMD:C_0402_1005Metric -> Capacitor_SMD:C_0603_1608Metric
- D10, D3, D4, D5, D9: footprint (none) -> LED_SMD:LED_0603_1608Metric
- J12: renamed from J13; footprint (none) -> Connector_Audio:Jack_3.5mm_CUI_SJ-3523-SMT_Horizontal
- J14: footprint (none) -> Connector_Card:microSD_HC_Wuerth_693072010801
- SW6: footprint Rotary_Encoder:RotaryEncoder_Alps_EC11E_Vertical_H20mm -> Rotary_Encoder:RotaryEncoder_Alps_EC11E-Switch_Vertical_H20mm
Connections:
- net SGND is gone; now on net GND: J12.S, U9.15 (SGND)
- net GND: now also C45.1, C49.1
- net GPIO23_A: now also R25.1; no longer D11.4 (DIN)
- net GPIO23_B: now also R26.1; no longer D14.4 (DIN)
- net VBUS_A: now also D1.1 (K)
- net VBUS_B: now also D2.1 (K)
- net at R19.2: now also U9.1 (INL-)
- net at R20.2: now also U9.4 (INR-)
- net at U9.2 (INL+): now also C49.2
- net at J3.A4 (VBUS), J3.A9 (VBUS), J3.B4 (VBUS)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: now also D1.2 (A), D2.2 (A)
- net at U9.3 (INR+): now also C45.2
- new net: D11.4 (DIN), R25.2
- new net: D14.4 (DIN), R26.2
- no-connect marks 6 -> 8
Other:
- moved on the sheet: C44, C50, C51, D11, D12, D13, D14, D15, D16, J12, U9

Commit message: 08062026 - wrapping up schematic work!
Parts:
- removed J6, J7, J8, J9: Conn_01x20, Connector_PinHeader_2.54mm:PinHeader_1x20_P2.54mm_Vertical, symbol Connector_Generic:Conn_01x20
- added J13, J25, J9: Conn_01x02, Connector_PinHeader_2.54mm:PinHeader_1x02_P2.54mm_Vertical, symbol Connector_Generic:Conn_01x02
- added J15, J17, J18, J19: Conn_01x03, Connector_PinHeader_2.54mm:PinHeader_1x03_P2.54mm_Vertical, symbol Connector_Generic:Conn_01x03
- added J16: Conn_01x06, Connector_PinHeader_2.54mm:PinHeader_1x06_P2.54mm_Vertical, symbol Connector_Generic:Conn_01x06
- added J20, J21, J6, J8: Conn_01x04, Connector_PinHeader_2.54mm:PinHeader_1x04_P2.54mm_Vertical, symbol Connector_Generic:Conn_01x04
- added J22, J23, J24: Conn_01x05, Connector_PinHeader_2.54mm:PinHeader_1x05_P2.54mm_Vertical, symbol Connector_Generic:Conn_01x05
- added J7: Conn_01x07, Connector_PinHeader_2.54mm:PinHeader_1x07_P2.54mm_Vertical, symbol Connector_Generic:Conn_01x07
Connections:
- net +3V3_A: now also J15.2 (Pin_2)
- net +3V3_B: now also J17.2 (Pin_2)
- net GND: now also J15.3 (Pin_3), J17.3 (Pin_3)
- net GPIO0_A: now also J6.1 (Pin_1)
- net GPIO0_B: now also J6.4 (Pin_4)
- net GPIO10_A: now also J7.7 (Pin_7)
- net GPIO10_B: now also J16.3 (Pin_3)
- net GPIO11_A: now also J8.1 (Pin_1)
- net GPIO11_B: now also J16.4 (Pin_4)
- net GPIO12_A: now also J8.2 (Pin_2)
- net GPIO12_B: now also J16.5 (Pin_5)
- net GPIO13_A: now also J8.3 (Pin_3)
- net GPIO13_B: now also J16.6 (Pin_6)
- net GPIO14_A: now also J8.4 (Pin_4)
- net GPIO14_B: now also J22.5 (Pin_5)
- net GPIO15_A: now also J21.1 (Pin_1)
- net GPIO15_B: now also J23.1 (Pin_1)
- net GPIO16_A: now also J9.1 (Pin_1)
- net GPIO16_B: now also J9.2 (Pin_2)
- net GPIO18_A: now also J13.1 (Pin_1)
- net GPIO18_B: now also J23.2 (Pin_2)
- net GPIO19_A: now also J13.2 (Pin_2)
- net GPIO19_B: now also J23.3 (Pin_3)
- net GPIO1_A: now also J6.2 (Pin_2)
- net GPIO20_A: now also J21.2 (Pin_2)
- net GPIO20_B: now also J23.4 (Pin_4)
- net GPIO21_A: now also J21.3 (Pin_3)
- net GPIO21_B: now also J23.5 (Pin_5)
- net GPIO22_A: now also J21.4 (Pin_4)
- net GPIO22_B: now also J24.1 (Pin_1)
- net GPIO23_A: now also J19.1 (Pin_1)
- net GPIO23_B: now also J18.1 (Pin_1)
- net GPIO24_A: now also J19.2 (Pin_2)
- net GPIO24_B: now also J18.2 (Pin_2)
- net GPIO25_A: now also J19.3 (Pin_3)
- net GPIO25_B: now also J18.3 (Pin_3)
- net GPIO26_C0_A: now also J20.1 (Pin_1)
- net GPIO26_C0_B: now also J24.2 (Pin_2)
- net GPIO27_C1_A: now also J20.2 (Pin_2)
- net GPIO27_C1_B: now also J24.3 (Pin_3)
- net GPIO28_C2_A: now also J20.3 (Pin_3)
- net GPIO28_C2_B: now also J24.4 (Pin_4)
- net GPIO29_C3_A: now also J20.4 (Pin_4)
- net GPIO29_C3_B: now also J24.5 (Pin_5)
- net GPIO2_A: now also J6.3 (Pin_3)
- net GPIO4_A: now also J7.1 (Pin_1)
- net GPIO4_B: now also J22.1 (Pin_1)
- net GPIO5_A: now also J7.2 (Pin_2)
- net GPIO5_B: now also J22.2 (Pin_2)
- net GPIO6_A: now also J7.3 (Pin_3)
- net GPIO6_B: now also J22.3 (Pin_3)
- net GPIO7_A: now also J7.4 (Pin_4)
- net GPIO7_B: now also J22.4 (Pin_4)
- net GPIO8_A: now also J7.5 (Pin_5)
- net GPIO8_B: now also J16.1 (Pin_1)
- net GPIO9_A: now also J7.6 (Pin_6)
- net GPIO9_B: now also J16.2 (Pin_2)
- net RUN_A: now also J25.1 (Pin_1)
- net RUN_B: now also J25.2 (Pin_2)
- net VBUS_A: now also J15.1 (Pin_1)
- net VBUS_B: now also J17.1 (Pin_1)
Other:
- note added: "TODO: NEED TO VERIFY DIODE SELECTION!!!"
- note removed: "TODO: NEED TO SELECT DIODES!!!"

Commit message: start pcb work! mcu_a wired!
Parts:
- C1, C10, C11, C12, C15, C16, C17, C2, C20, C21, C22, C23, C24, C25, C26, C27, C28, C29, C3, C30, C31, C32, C33, C34, C35, C36, C37, C38, C39, C4, C40, C41, C42, C43, C44, C45, C46, C47, C48, C49, C5, C50, C51, C6, C7, C8, C9: footprint Capacitor_SMD:C_0603_1608Metric -> Capacitor_SMD:C_0402_1005Metric
- U3, U6: value W25Q128JVS -> W25Q16JVZPIQ TR; footprint Package_SO:SOIC-8_5.23x5.23mm_P1.27mm -> Package_SON:Winbond_USON-8-1EP_3x2mm_P0.5mm_EP0.2x1.6mm
Changed lines of the file:
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@@
 			)
 		)
-		(property "Footprint" "Capacitor_SMD:C_0603_1608Metric"
+		(property "Footprint" "Capacitor_SMD:C_0402_1005Metric"
 			(at 394.0048 209.55 0)
 			(effects
@@
 			)
 		)
-		(property "Footprint" "Capacitor_SMD:C_0603_1608Metric"
+		(property "Footprint" "Capacitor_SMD:C_0402_1005Metric"
 			(at 293.0652 177.8 0)
 			(effects
@@
 			)
 		)
-		(property "Footprint" "Capacitor_SMD:C_0603_1608Metric"
+		(property "Footprint" "Capacitor_SMD:C_0402_1005Metric"
 			(at 158.4452 33.02 0)
 			(effects
@@
 			)
 		)
-		(property "Footprint" "Capacitor_SMD:C_0603_1608Metric"
+		(property "Footprint" "Capacitor_SMD:C_0402_1005Metric"
 			(at 145.7452 33.02 0)
 			(effects
@@
 			)
 		)
-		(property "Footprint" "Capacitor_SMD:C_0603_1608Metric"
+		(property "Footprint" "Capacitor_SMD:C_0402_1005Metric"
 			(at 336.8548 222.25 0)
 			(effects
@@
 			)
 		)
-		(property "Footprint" "Capacitor_SMD:C_0603_1608Metric"
+		(property "Footprint" "Capacitor_SMD:C_0402_1005Metric"
 			(at 103.8352 144.78 0)
 			(effects
@@
 			)
 		)
-		(property "Footprint" "Capacitor_SMD:C_0603_1608Metric"
+		(property "Footprint" "Capacitor_SMD:C_0402_1005Metric"
 			(at 115.2652 33.02 0)
 			(effects
@@
 			)
 		)
-		(property "Footprint" "Capacitor_SMD:C_0603_1608Metric"
+		(property "Footprint" "Capacitor_SMD:C_0402_1005Metric"
 			(at 146.05 165.4048 0)
 			(effects
@@
 			)
 		)
-		(property "Footprint" "Capacitor_SMD:C_0603_1608Metric"
+		(property "Footprint" "Capacitor_SMD:C_0402_1005Metric"
 			(at 183.8452 144.78 0)
 			(effects
@@
 			)
 		)
-		(property "Footprint" "Capacitor_SMD:C_0603_1608Metric"
+		(property "Footprint" "Capacitor_SMD:C_0402_1005Metric"
 			(at 334.3148 204.47 0)
 			(effects
@@
 			)
 		)
-		(property "Footprint" "Capacitor_SMD:C_0603_1608Metric"
+		(property "Footprint" "Capacitor_SMD:C_0402_1005Metric"
 			(at 304.4952 177.8 0)
 			(effects
@@
 			)
 		)
-		(property "Footprint" "Capacitor_SMD:C_0603_1608Metric"
+		(property "Footprint" "Capacitor_SMD:C_0402_1005Metric"
 			(at 298.1452 177.8 0)
 			(effects
@@
 			)
 		)
-		(property "Footprint" "Capacitor_SMD:C_0603_1608Metric"
+		(property "Footprint" "Capacitor_SMD:C_0402_1005Metric"
 			(at 152.0952 144.78 0)
 			(effects
@@
 			)
 		)
-		(property "Footprint" "Capacitor_SMD:C_0603_1608Metric"
+		(property "Footprint" "Capacitor_SMD:C_0402_1005Metric"
 			(at 365.76 223.2152 0)
 			(effects
@@
 			)
 		)
-		(property "Footprint" "Capacitor_SMD:C_0603_1608Metric"
+		(property "Footprint" "Capacitor_SMD:C_0402_1005Metric"
 			(at 171.1452 144.78 0)
 			(effects
@@
 			)
 		)
-		(property "Footprint" "Capacitor_SMD:C_0603_1608Metric"
+		(property "Footprint" "Capacitor_SMD:C_0402_1005Metric"
 			(at 133.0452 33.02 0)
 			(effects
@@
 			)
 		)
-		(property "Footprint" "Capacitor_SMD:C_0603_1608Metric"
+		(property "Footprint" "Capacitor_SMD:C_0402_1005Metric"
 			(at 145.7452 144.78 0)
 			(effects
@@
 			)
 		)
-		(property "Footprint" "Capacitor_SMD:C_0603_1608Metric"
+		(property "Footprint" "Capacitor_SMD:C_0402_1005Metric"
 			(at 177.4952 33.02 0)
 			(effects
@@
 			)
 		)
-		(property "Footprint" "Capacitor_SMD:C_0603_1608Metric"
+		(property "Footprint" "Capacitor_SMD:C_0402_1005Metric"
 			(at 164.7952 33.02 0)
 			(effects
@@
 			)
 		)
-		(property "Footprint" "Capacitor_SMD:C_0603_1608Metric"
+		(property "Footprint" "Capacitor_SMD:C_0402_1005Metric"
 			(at 332.4352 177.8 0)
 			(effects
@@
 			)
 		)
-		(property "Footprint" "Capacitor_SMD:C_0603_1608Metric"
+		(property "Footprint" "Capacitor_SMD:C_0402_1005Metric"
 			(at 326.0852 177.8 0)
 			(effects
@@
 			)
 		)
-		(property "Footprint" "Capacitor_SMD:C_0603_1608Metric"
+		(property "Footprint" "Capacitor_SMD:C_0402_1005Metric"
 			(at 108.9152 144.78 0)
 			(effects
@@
 			)
 		)
-		(property "Footprint" "Capacitor_SMD:C_0603_1608Metric"
+		(property "Footprint" "Capacitor_SMD:C_0402_1005Metric"
 			(at 183.8452 33.02 0)
 			(effects
@@
 			)
 		)
-		(property "Footprint" "Capacitor_SMD:C_0603_1608Metric"
+		(property "Footprint" "Capacitor_SMD:C_0402_1005Metric"
 			(at 146.05 53.6448 0)
 			(effects
@@
 			)
 		)
-		(property "Value" "W25Q128JVS"
+		(property "Value" "W25Q16JVZPIQ TR"
 			(at 143.51 79.502 90)
 			(effects
@@
 			)
 		)
-		(property "Footprint" "Package_SO:SOIC-8_5.23x5.23mm_P1.27mm"
+		(property "Footprint" "Package_SON:Winbond_USON-8-1EP_3x2mm_P0.5mm_EP0.2x1.6mm"
 			(at 137.16 46.99 0)
 			(effects
@@
 			)
 		)
-		(property "Datasheet" "https://www.winbond.com/resource-files/w25q128jv_dtr%20revc%2003272018%20plus.pdf"
+		(property "Datasheet" ""
 			(at 137.16 44.45 0)
 			(effects
@@
 			)
 		)
-		(property "Description" "128Mb Serial Flash Memory, Standard/Dual/Quad SPI, SOIC-8"
+		(property "Description" ""
 			(at 137.16 41.91 0)
 			(effects
@@
 			)
 		)
-		(property "Value" "W25Q128JVS"
+		(property "Value" "W25Q16JVZPIQ TR"
 			(at 143.51 191.262 90)
 			(effects
@@
 			)
 		)
-		(property "Footprint" "Package_SO:SOIC-8_5.23x5.23mm_P1.27mm"
+		(property "Footprint" "Package_SON:Winbond_USON-8-1EP_3x2mm_P0.5mm_EP0.2x1.6mm"
 			(at 137.16 158.75 0)
 			(effects
@@
 			)
 		)
-		(property "Datasheet" "https://www.winbond.com/resource-files/w25q128jv_dtr%20revc%2003272018%20plus.pdf"
+		(property "Datasheet" ""
 			(at 137.16 156.21 0)
 			(effects
@@
 			)
 		)
-		(property "Description" "128Mb Serial Flash Memory, Standard/Dual/Quad SPI, SOIC-8"
+		(property "Description" ""
 			(at 137.16 153.67 0)
 			(effects
@@
 			)
 		)
-		(property "Footprint" "Capacitor_SMD:C_0603_1608Metric"
+		(property "Footprint" "Capacitor_SMD:C_0402_1005Metric"
 			(at 177.4952 144.78 0)
 			(effects
@@
 			)
 		)
-		(property "Footprint" "Capacitor_SMD:C_0603_1608Metric"
+		(property "Footprint" "Capacitor_SMD:C_0402_1005Metric"
 			(at 109.22 101.9048 0)
 			(effects
@@
 			)
 		)
-		(property "Footprint" "Capacitor_SMD:C_0603_1608Metric"
+		(property "Footprint" "Capacitor_SMD:C_0402_1005Metric"
 			(at 108.9152 33.02 0)
 			(effects
@@
 			)
 		)
-		(property "Footprint" "Capacitor_SMD:C_0603_1608Metric"
+		(property "Footprint" "Capacitor_SMD:C_0402_1005Metric"
 			(at 63.8048 214.63 0)
 			(effects
@@
 			)
 		)
-		(property "Footprint" "Capacitor_SMD:C_0603_1608Metric"
+		(property "Footprint" "Capacitor_SMD:C_0402_1005Metric"
 			(at 133.0452 144.78 0)
 			(effects
@@
 			)
 		)
-		(property "Footprint" "Capacitor_SMD:C_0603_1608Metric"
+		(property "Footprint" "Capacitor_SMD:C_0402_1005Metric"
 			(at 139.3952 33.02 0)
 			(effects
@@
 			)
 		)
-		(property "Footprint" "Capacitor_SMD:C_0603_1608Metric"
+		(property "Footprint" "Capacitor_SMD:C_0402_1005Metric"
 			(at 45.4152 214.63 0)
 			(effects
@@
 			)
 		)
-		(property "Footprint" "Capacitor_SMD:C_0603_1608Metric"
+		(property "Footprint" "Capacitor_SMD:C_0402_1005Metric"
 			(at 158.4452 144.78 0)
 			(effects
@@
 			)
 		)
-		(property "Footprint" "Capacitor_SMD:C_0603_1608Metric"
+		(property "Footprint" "Capacitor_SMD:C_0402_1005Metric"
 			(at 152.0952 33.02 0)
 			(effects
@@
 			)
 		)
-		(property "Footprint" "Capacitor_SMD:C_0603_1608Metric"
+		(property "Footprint" "Capacitor_SMD:C_0402_1005Metric"
 			(at 397.2052 104.14 0)
 			(effects
@@
 			)
 		)
-		(property "Footprint" "Capacitor_SMD:C_0603_1608Metric"
+		(property "Footprint" "Capacitor_SMD:C_0402_1005Metric"
 			(at 171.1452 33.02 0)
 			(effects
@@
 			)
 		)
-		(property "Footprint" "Capacitor_SMD:C_0603_1608Metric"
+		(property "Footprint" "Capacitor_SMD:C_0402_1005Metric"
 			(at 360.68 178.1048 0)
 			(effects
@@
 			)
 		)
-		(property "Footprint" "Capacitor_SMD:C_0603_1608Metric"
+		(property "Footprint" "Capacitor_SMD:C_0402_1005Metric"
 			(at 396.24 181.9148 0)
 			(effects
@@
 			)
 		)
-		(property "Footprint" "Capacitor_SMD:C_0603_1608Metric"
+		(property "Footprint" "Capacitor_SMD:C_0402_1005Metric"
 			(at 115.2652 144.78 0)
 			(effects
@@
 			)
 		)
-		(property "Footprint" "Capacitor_SMD:C_0603_1608Metric"
+		(property "Footprint" "Capacitor_SMD:C_0402_1005Metric"
 			(at 164.7952 144.78 0)
 			(effects
@@
 			)
 		)
-		(property "Footprint" "Capacitor_SMD:C_0603_1608Metric"
+		(property "Footprint" "Capacitor_SMD:C_0402_1005Metric"
 			(at 109.22 223.8248 0)
 			(effects
@@
 			)
 		)
-		(property "Footprint" "Capacitor_SMD:C_0603_1608Metric"
+		(property "Footprint" "Capacitor_SMD:C_0402_1005Metric"
 			(at 109.22 213.6648 0)
 			(effects
@@
 			)
 		)
-		(property "Footprint" "Capacitor_SMD:C_0603_1608Metric"
+		(property "Footprint" "Capacitor_SMD:C_0402_1005Metric"
 			(at 360.68 174.9552 0)
 			(effects
@@
 			)
 		)
-		(property "Footprint" "Capacitor_SMD:C_0603_1608Metric"
+		(property "Footprint" "Capacitor_SMD:C_0402_1005Metric"
 			(at 109.22 112.0648 0)
 			(effects
@@
 			)
 		)
-		(property "Footprint" "Capacitor_SMD:C_0603_1608Metric"
+		(property "Footprint" "Capacitor_SMD:C_0402_1005Metric"
 			(at 333.7052 222.25 0)
 			(effects
@@
 			)
 		)
-		(property "Footprint" "Capacitor_SMD:C_0603_1608Metric"
+		(property "Footprint" "Capacitor_SMD:C_0402_1005Metric"
 			(at 309.5752 177.8 0)
 			(effects
@@
 			)
 		)
-		(property "Footprint" "Capacitor_SMD:C_0603_1608Metric"
+		(property "Footprint" "Capacitor_SMD:C_0402_1005Metric"
 			(at 139.3952 144.78 0)
 			(effects
@@
 			)
 		)
-		(property "Footprint" "Capacitor_SMD:C_0603_1608Metric"
+		(property "Footprint" "Capacitor_SMD:C_0402_1005Metric"
 			(at 102.5652 33.02 0)
 			(effects

Commit message: 08162026 - start pcb! (layout and both mcus wired!)
Changed lines of the file:
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@@
 	)
 	(junction
-		(at 102.87 144.78)
-		(diameter 0)
-		(color 0 0 0 0)
-	)
-	(junction
 		(at 331.47 177.8)
 		(diameter 0)
@@
 	)
 	(junction
-		(at 102.87 137.16)
-		(diameter 0)
-		(color 0 0 0 0)
-	)
-	(junction
 		(at 114.3 33.02)
 		(diameter 0)
@@
 	(wire
 		(pts
-			(xy 101.6 137.16) (xy 102.87 137.16)
-		)
-		(stroke
-			(width 0)
-			(type default)
-		)
-	)
-	(wire
-		(pts
 			(xy 151.13 33.02) (xy 157.48 33.02)
 		)
@@
 		)
 		(stroke
-			(width 0)
-			(type default)
-		)
-	)
-	(wire
-		(pts
-			(xy 101.6 144.78) (xy 102.87 144.78)
-		)
-		(stroke
