File: pcb/board/board.kicad_sch (KiCad schematic)
At the start: 129 parts, among them J1 (A) USB_C_Receptacle_USB2.0_1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, J10 OLED_128x32, J11 LCD_128x160, J12 AudioJack3, J13 Conn_01x01, J14 Micro_SD_Card, J15 Conn_01x01, J16 Conn_01x01, J17 Conn_01x01, J18 Conn_01x01, J19 Conn_01x01, J2 (B) USB_C_Receptacle_USB2.0_1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, J20 Conn_01x01, J21 Conn_01x01, J22 Conn_01x01, J3 (C) USB_C_Receptacle_USB2.0_1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, J4 Conn_01x03, J5 Conn_01x03, J6 Conn_01x01, J7 Conn_01x01, J8 Conn_01x01, J9 Conn_01x01, SW1 SW_Push, SW2 SW_Push, SW3 Switch, SW4 Switch, SW5 Switch, SW6 RotaryEncoder_Switch, U1 RP2040, U2 NCP1117-3.3_SOT223, U3 W25Q16JVZPIQ TR, U4 NCP1117-3.3_SOT223, U5 RP2040, U6 W25Q16JVZPIQ TR, U7 PCM5101A, U8 TLV70033_SOT23-5, U9 TPA6132A2RTE, Y1 12MHz, Y2 12MHz

Commit message: more ground vias and some silkscreen text fixes!
Parts:
- added C52: 2.2uF, Capacitor_SMD:C_0402_1005Metric, symbol Device:C
Connections:
- net +3V3_AUDIO: now also C52.1
- net GND: now also C52.2
Other:
- note removed: "TODO: DOUBLE CHECK AMP POWER!!!"
- moved on the sheet: C44, J12
Changed lines of the file:
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@@
 	)
 	(junction
+		(at 374.65 180.34)
+		(diameter 0)
+		(color 0 0 0 0)
+	)
+	(junction
 		(at 134.62 260.35)
 		(diameter 0)
@@
 	)
 	(junction
+		(at 398.78 182.88)
+		(diameter 0)
+		(color 0 0 0 0)
+	)
+	(junction
 		(at 170.18 137.16)
 		(diameter 0)
@@
 	(wire
 		(pts
-			(xy 401.32 171.45) (xy 401.32 191.77)
+			(xy 401.32 170.18) (xy 401.32 191.77)
 		)
 		(stroke
@@
 	(wire
 		(pts
-			(xy 397.51 182.88) (xy 396.24 182.88)
+			(xy 398.78 182.88) (xy 394.97 182.88)
 		)
 		(stroke
@@
 	(wire
 		(pts
-			(xy 401.32 171.45) (xy 392.43 171.45)
+			(xy 401.32 170.18) (xy 397.51 170.18)
 		)
 		(stroke
@@
 	(wire
 		(pts
-			(xy 397.51 184.15) (xy 397.51 182.88)
+			(xy 398.78 182.88) (xy 398.78 184.15)
 		)
 		(stroke
@@
 	(wire
 		(pts
-			(xy 397.51 173.99) (xy 392.43 173.99)
+			(xy 398.78 172.72) (xy 397.51 172.72)
 		)
 		(stroke
@@
 	(wire
 		(pts
+			(xy 398.78 180.34) (xy 387.35 180.34)
+		)
+		(stroke
+			(width 0)
+			(type default)
+		)
+	)
+	(wire
+		(pts
 			(xy 266.7 48.26) (xy 265.43 48.26)
 		)
@@
 	(wire
 		(pts
+			(xy 374.65 180.34) (xy 379.73 180.34)
+		)
+		(stroke
+			(width 0)
+			(type default)
+		)
+	)
+	(wire
+		(pts
 			(xy 204.47 154.94) (xy 205.74 154.94)
 		)
@@
 	(wire
 		(pts
-			(xy 374.65 182.88) (xy 374.65 184.15)
-		)
-		(stroke
-			(width 0)
-			(type default)
-		)
-	)
-	(wire
-		(pts
 			(xy 125.73 184.15) (xy 127 184.15)
 		)
@@
 	(wire
 		(pts
+			(xy 398.78 180.34) (xy 398.78 182.88)
+		)
+		(stroke
+			(width 0)
+			(type default)
+		)
+	)
+	(wire
+		(pts
 			(xy 44.45 24.13) (xy 53.34 24.13)
 		)
@@
 	(wire
 		(pts
-			(xy 377.19 182.88) (xy 388.62 182.88)
+			(xy 377.19 182.88) (xy 387.35 182.88)
 		)
 		(stroke
@@
 	(wire
 		(pts
+			(xy 374.65 179.07) (xy 374.65 180.34)
+		)
+		(stroke
+			(width 0)
+			(type default)
+		)
+	)
+	(wire
+		(pts
 			(xy 332.74 212.09) (xy 332.74 214.63)
 		)
@@
 	(wire
 		(pts
-			(xy 402.59 168.91) (xy 402.59 196.85)
+			(xy 402.59 167.64) (xy 402.59 196.85)
 		)
 		(stroke
@@
 	(wire
 		(pts
-			(xy 392.43 168.91) (xy 402.59 168.91)
+			(xy 397.51 167.64) (xy 402.59 167.64)
 		)
 		(stroke
@@
 	(wire
 		(pts
+			(xy 374.65 180.34) (xy 374.65 184.15)
+		)
+		(stroke
+			(width 0)
+			(type default)
+		)
+	)
+	(wire
+		(pts
 			(xy 212.09 276.86) (xy 210.82 276.86)
 		)
@@
 	(wire
 		(pts
-			(xy 397.51 175.26) (xy 397.51 173.99)
+			(xy 398.78 173.99) (xy 398.78 172.72)
 		)
 		(stroke
@@
 		)
 	)
-	(text "TODO: DOUBLE CHECK\nAMP POWER!!!"
-		(exclude_from_sim no)
-		(at 356.87 260.604 0)
-		(effects
-			(font
-				(size 3.81 3.81)
-			)
-		)
-	)
 	(text "0-3: SPI0 MCU\n8-13: LCD 128x160 Display\n16-17: UART0 MCU (backup)\n23-25: RGB, Board, Boot LEDS"
 		(exclude_from_sim no)
@@
 	(symbol
 		(lib_id "power:GND")
-		(at 397.51 184.15 0)
+		(at 398.78 184.15 0)
 		(unit 1)
 		(exclude_from_sim no)
@@
 		(fields_autoplaced yes)
 		(property "Reference" "#PWR069"
-			(at 397.51 190.5 0)
+			(at 398.78 190.5 0)
 			(effects
 				(font
@@
 		)
 		(property "Value" "GND"
-			(at 397.51 189.23 0)
+			(at 398.78 189.23 0)
 			(effects
 				(font
@@
 		)
 		(property "Footprint" ""
-			(at 397.51 184.15 0)
+			(at 398.78 184.15 0)
 			(effects
 				(font
@@
 		)
 		(property "Datasheet" ""
-			(at 397.51 184.15 0)
+			(at 398.78 184.15 0)
 			(effects
 				(font
@@
 		)
 		(property "Description" "Power symbol creates a global label with name \"GND\" , ground"
-			(at 397.51 184.15 0)
+			(at 398.78 184.15 0)
 			(effects
 				(font
@@
 	(symbol
 		(lib_id "Connector_Audio:AudioJack3")
-		(at 387.35 171.45 0)
+		(at 392.43 170.18 0)
 		(mirror x)
 		(unit 1)
@@
 		(dnp no)
 		(property "Reference" "J12"
-			(at 397.002 164.846 0)
+			(at 402.082 163.576 0)
 			(effects
 				(font
@@
 		)
 		(property "Value" "AudioJack3"
-			(at 392.684 164.846 0)
+			(at 397.764 163.576 0)
 			(effects
 				(font
@@
 		)
 		(property "Footprint" "Connector_Audio:Jack_3.5mm_CUI_SJ-3523-SMT_Horizontal"
-			(at 387.35 171.45 0)
+			(at 392.43 170.18 0)
 			(effects
 				(font
@@
 		)
 		(property "Datasheet" "~"
-			(at 387.35 171.45 0)
+			(at 392.43 170.18 0)
 			(effects
 				(font
@@
 		)
 		(property "Description" "Audio Jack, 3 Poles (Stereo / TRS)"
-			(at 387.35 171.45 0)
+			(at 392.43 170.18 0)
 			(effects
 				(font
@@
 	(symbol
 		(lib_id "power:+3V3")
-		(at 374.65 182.88 0)
+		(at 374.65 179.07 0)
 		(unit 1)
 		(exclude_from_sim no)
@@
 		(dnp no)
 		(property "Reference" "#PWR097"
-			(at 374.65 186.69 0)
+			(at 374.65 182.88 0)
 			(effects
 				(font
@@
 		)
 		(property "Value" "+3V3_AUDIO"
-			(at 368.554 177.8 0)
+			(at 368.554 173.99 0)
 			(effects
 				(font
@@
 		)
 		(property "Footprint" ""
-			(at 374.65 182.88 0)
+			(at 374.65 179.07 0)
 			(effects
 				(font
@@
 		)
 		(property "Datasheet" ""
-			(at 374.65 182.88 0)
+			(at 374.65 179.07 0)
 			(effects
 				(font
@@
 		)
 		(property "Description" "Power symbol creates a global label with name \"+3V3\""
-			(at 374.65 182.88 0)
+			(at 374.65 179.07 0)
 			(effects
 				(font
@@
 	(symbol
 		(lib_id "power:GND")
-		(at 397.51 175.26 0)
+		(at 398.78 173.99 0)
 		(unit 1)
 		(exclude_from_sim no)
@@
 		(fields_autoplaced yes)
 		(property "Reference" "#PWR070"
-			(at 397.51 181.61 0)
+			(at 398.78 180.34 0)
 			(effects
 				(font
@@
 		)
 		(property "Value" "GND"
-			(at 397.51 180.34 0)
+			(at 398.78 179.07 0)
 			(effects
 				(font
@@
 		)
 		(property "Footprint" ""
-			(at 397.51 175.26 0)
+			(at 398.78 173.99 0)
 			(effects
 				(font
@@
 		)
 		(property "Datasheet" ""
-			(at 397.51 175.26 0)
+			(at 398.78 173.99 0)
 			(effects
 				(font
@@
 		)
 		(property "Description" "Power symbol creates a global label with name \"GND\" , ground"
-			(at 397.51 175.26 0)
+			(at 398.78 173.99 0)
 			(effects
 				(font
@@
 	(symbol
 		(lib_id "Device:C")
-		(at 392.43 182.88 90)
+		(at 391.16 182.88 90)
 		(unit 1)
 		(exclude_from_sim no)
@@
 		(dnp no)
 		(property "Reference" "C44"
-			(at 394.462 188.976 90)
+			(at 393.192 188.976 90)
 			(effects
 				(font
@@
 		)
 		(property "Value" "2.2uF"
-			(at 395.224 186.69 90)
+			(at 393.954 186.69 90)
 			(effects
 				(font
@@
 		)
 		(property "Footprint" "Capacitor_SMD:C_0402_1005Metric"
-			(at 396.24 181.9148 0)
+			(at 394.97 181.9148 0)
 			(effects
 				(font
@@
 		)
 		(property "Datasheet" "~"
-			(at 392.43 182.88 0)
+			(at 391.16 182.88 0)
 			(effects
 				(font
@@
 		)
 		(property "Description" "Unpolarized capacitor"
-			(at 392.43 182.88 0)
+			(at 391.16 182.88 0)
 			(effects
 				(font
@@
 					(unit 1)
 				)
+			)
+		)
+	)
+	(symbol
+		(lib_id "Device:C")
+		(at 383.54 180.34 90)
+		(mirror x)
+		(unit 1)
+		(exclude_from_sim no)
+		(in_bom yes)
+		(on_board yes)
+		(dnp no)
+		(property "Reference" "C52"
+			(at 385.572 174.244 90)
+			(effects
+				(font
+					(size 1.27 1.27)
+				)
+				(justify left)
+			)
+		)
+		(property "Value" "2.2uF"
+			(at 386.334 176.53 90)
+			(effects
+				(font
+					(size 1.27 1.27)
+				)
+				(justify left)
+			)
+		)
+		(property "Footprint" "Capacitor_SMD:C_0402_1005Metric"
+			(at 387.35 181.3052 0)
+			(effects
+				(font
+					(size 1.27 1.27)
+				)
+				(hide yes)
+			)
+		)
+		(property "Datasheet" "~"
+			(at 383.54 180.34 0)
+			(effects
+				(font
+					(size 1.27 1.27)
+				)
+				(hide yes)
+			)
+		)
+		(property "Description" "Unpolarized capacitor"
+			(at 383.54 180.34 0)
+			(effects
+				(font
+					(size 1.27 1.27)
+				)
+				(hide yes)
+			)
+		)
+		(pin "1"
+		)
+		(pin "2"
+		)
+		(instances
+			(project "board"
+				(path "/ad83e94c-cf92-4843-8895-58faef287199"
+					(reference "C52")
+					(unit 1)
+				)
