File: pcb/board/board.kicad_pcb (KiCad board)
At the start: 2 copper layers, 56 x 80 mm, 132 parts, among them J1 (A) USB_C_Receptacle_USB2.0_1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, J10 OLED_128x32, J11 LCD_128x160, J12 AudioJack3, J13 Conn_01x02, J14 Micro_SD_Card, J15 Conn_01x03, J16 Conn_01x06, J17 Conn_01x03, J18 Conn_01x03, J19 Conn_01x03, J2 (B) USB_C_Receptacle_USB2.0_1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, J20 Conn_01x04, J21 Conn_01x04, J22 Conn_01x05, J23 Conn_01x05, J24 Conn_01x05, J25 Conn_01x02, J3 (C) USB_C_Receptacle_USB2.0_1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, J4 Conn_01x03, J5 Conn_01x03, J6 Conn_01x04, J7 Conn_01x07, J8 Conn_01x04, J9 Conn_01x02, SW1 SW_Push, SW2 SW_Push, SW3 Switch, SW4 Switch, SW5 Switch, SW6 RotaryEncoder_Switch, U1 RP2040, U2 NCP1117-3.3_SOT223, U3 W25Q16JVZPIQ TR, U4 NCP1117-3.3_SOT223, U5 RP2040, U6 W25Q16JVZPIQ TR, U7 PCM5101A, U8 TLV70033_SOT23-5, U9 TPA6132A2RTE, Y1 12MHz, Y2 12MHz

Commit message: 08162026 - start pcb! (layout and both mcus wired!)
Parts:
- C18, C19, D11, D12, D13, D14, D15, D16, J12, R8, R9, U8: moved to B.Cu
- moved U8 263.8 mm to (134.8, 67.2)
- moved C18 234.4 mm to (106.2, 61.0), turned to 180 degrees
- moved C19 234.3 mm to (112.0, 72.0)
- moved J12 208.1 mm to (210.9, 96.9), turned to -90 degrees
- moved R14 187.4 mm to (126.8, 72.2)
- moved R15 184.9 mm to (120.2, 70.2), turned to 0 degrees
- moved R16 184.6 mm to (117.5, 86.2), turned to 0 degrees
- moved D4 181.3 mm to (109.0, 80.8), turned to 0 degrees
- moved D10 180.3 mm to (109.0, 82.8), turned to 0 degrees
- moved R12 178.7 mm to (117.3, 75.2), turned to -90 degrees
- moved R13 177.4 mm to (116.2, 75.2), turned to 90 degrees
- moved R9 176.2 mm to (112.2, 60.1), turned to 180 degrees
- moved R23 175.7 mm to (106.2, 82.8)
- moved R18 171.7 mm to (106.2, 80.8)
- moved R8 171.4 mm to (108.2, 60.8), turned to -90 degrees
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Routing:
- net +3V3_B: track 0.00 -> 69.5 mm, vias 0 -> 5
- net +1V1_B: track 0.00 -> 22.1 mm
- net USB_B D+: track 2.99 -> 25.1 mm
- net USB_B D-: track 2.99 -> 25.1 mm
- net QSPI_SS_B: track 0.00 -> 14.8 mm
- net VBUS_B: track 13.8 -> 25.2 mm, vias 0 -> 2
- net VBUS_A: track 23.7 -> 33.4 mm
- net XIN_B: track 0.00 -> 7.43 mm
- net QSPI_SD1_B: track 0.00 -> 6.98 mm
- net +3V3_A: track 69.6 -> 76.2 mm, vias 5 -> 7
- net QSPI_SD2_B: track 0.00 -> 5.53 mm
- net QSPI_SD3_B: track 0.00 -> 5.38 mm
- net QSPI_SCLK_B: track 0.00 -> 4.68 mm
- net QSPI_SD0_B: track 0.00 -> 3.74 mm
- net Net-(C22-Pad2): track 0.00 -> 3.48 mm
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
Commit message: audio stuff wired together!
Parts:
- C35, C36, C37, C38, C39, C40, C41, C42, C43, C44, C45, C46, C47, C49, C50, C51, R19, R20, U7, U9: moved to B.Cu
- J12: moved to F.Cu
- moved U7 311.8 mm to (30.8, 100.8), turned to 180 degrees
- moved R20 302.0 mm to (39.2, 101.8)
- moved R19 300.8 mm to (39.2, 104.8)
- moved C43 296.1 mm to (25.9, 99.1), turned to 180 degrees
- moved C40 294.7 mm to (25.9, 96.5), turned to 180 degrees
- moved C39 293.8 mm to (25.9, 97.5), turned to 180 degrees
- moved U9 291.5 mm to (42.5, 103.2)
- moved C41 285.7 mm to (35.2, 99.1), turned to -90 degrees
- moved C42 285.2 mm to (36.2, 100.0), turned to 90 degrees
- moved C49 282.5 mm to (39.2, 103.8)
- moved C36 282.0 mm to (36.2, 96.5)
- moved C38 282.0 mm to (35.8, 103.8)
- moved C37 281.6 mm to (35.8, 102.8)
- moved C35 281.2 mm to (36.2, 97.5)
- moved C45 280.4 mm to (39.2, 102.8)
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Routing:
- net GPIO4_A: track 0.00 -> 38.2 mm
- net GPIO5_A: track 0.00 -> 21.1 mm
- net GPIO13_A: track 0.00 -> 12.9 mm, vias 0 -> 1
- net +3V3_AUDIO: track 0.00 -> 12.5 mm, vias 0 -> 2
- net GPIO14_A: track 0.00 -> 11.2 mm, vias 0 -> 1
- net GPIO12_A: track 0.00 -> 10.0 mm, vias 0 -> 1
- net GPIO11_A: track 0.00 -> 8.98 mm, vias 0 -> 1
- net Net-(U7-OUTL): track 0.00 -> 8.11 mm
- net Net-(U7-OUTR): track 0.00 -> 5.14 mm, vias 0 -> 2
- net Net-(U7-VNEG): track 0.00 -> 2.66 mm
- net +3V3_A: track 76.2 -> 78.8 mm
- net Net-(U9-HPVSS): track 0.00 -> 2.06 mm
- net Net-(U7-CAPP): track 0.00 -> 1.71 mm
- net Net-(U7-CAPM): track 0.00 -> 1.71 mm
- net Net-(U9-INR-): track 0.00 -> 1.61 mm
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
Commit message: 08172026 - pcb work continues! (audio and most mcu pin connections!)
Parts:
- removed J13: Conn_01x02, Connector_PinHeader_2.54mm:PinHeader_1x02_P2.54mm_Vertical
- removed J16: Conn_01x06, Connector_PinHeader_2.54mm:PinHeader_1x06_P2.54mm_Vertical
- removed J18, J19: Conn_01x03, Connector_PinHeader_2.54mm:PinHeader_1x03_P2.54mm_Vertical
- removed J20, J21, J8: Conn_01x04, Connector_PinHeader_2.54mm:PinHeader_1x04_P2.54mm_Vertical
- removed J22, J23, J24: Conn_01x05, Connector_PinHeader_2.54mm:PinHeader_1x05_P2.54mm_Vertical
- removed J7: Conn_01x07, Connector_PinHeader_2.54mm:PinHeader_1x07_P2.54mm_Vertical
- D5, R24: moved to F.Cu
- moved J17 153.2 mm to (194.0, 75.2)
- moved C39 110.4 mm to (134.2, 76.2), turned to 0 degrees
- moved C40 110.4 mm to (134.2, 75.2), turned to 0 degrees
- moved C43 109.0 mm to (132.4, 75.9), turned to 90 degrees
- moved U7 102.0 mm to (130.8, 80.8), turned to 90 degrees
- moved C35 100.0 mm to (135.2, 83.8)
- moved C36 100.0 mm to (135.2, 82.8)
- moved J25 99.3 mm to (162.5, 80.2)
- moved C41 98.1 mm to (132.4, 85.2), turned to 180 degrees
- moved C42 96.2 mm to (131.5, 86.2), turned to 0 degrees
- moved C37 94.5 mm to (128.8, 85.8), turned to -90 degrees
- moved C38 93.7 mm to (127.8, 85.8), turned to -90 degrees
- moved R20 91.4 mm to (129.8, 89.2), turned to -90 degrees
- moved C45 90.5 mm to (128.8, 89.2), turned to -90 degrees
- moved C49 89.7 mm to (127.8, 89.2), turned to -90 degrees
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Connections:
- U9 pad 13: GPIO29_C3_A -> GPIO20_A
- U9 pad 6: GPIO21_A -> GPIO22_A
- U9 pad 7: GPIO22_A -> GPIO21_A
Routing:
- net GPIO18_A: track 0.00 -> 60.2 mm, vias 0 -> 2
- net GPIO19_A: track 0.00 -> 57.1 mm, vias 0 -> 1
- net GPIO6_A: track 0.00 -> 44.9 mm, vias 0 -> 2
- net GPIO4_A: track 38.2 -> 81.4 mm, vias 0 -> 2
- net +3V3_A: track 78.8 -> 118.9 mm, vias 7 -> 10
- net GPIO5_A: track 21.1 -> 60.1 mm, vias 0 -> 2
- net GPIO16_A: track 0.00 -> 37.1 mm, vias 0 -> 2
- net GPIO16_B: track 0.00 -> 37.0 mm, vias 0 -> 2
- net Net-(U9-OUTL): track 0.00 -> 35.7 mm, vias 0 -> 1
- net GPIO9_A: track 0.00 -> 31.5 mm
- net +3V3_AUDIO: track 12.5 -> 43.1 mm, vias 2 -> 4
- net GPIO0_B: track 0.00 -> 29.4 mm, vias 0 -> 2
- net GPIO13_B: track 0.00 -> 29.3 mm, vias 0 -> 3
- net GPIO0_A: track 0.00 -> 28.9 mm, vias 0 -> 2
- net GPIO10_B: track 0.00 -> 28.8 mm, vias 0 -> 1
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
Commit message: leds and more connections!
Parts:
- removed J17, J4, J5: Conn_01x03, Connector_PinHeader_2.54mm:PinHeader_1x03_P2.54mm_Vertical
- removed J25, J9: Conn_01x02, Connector_PinHeader_2.54mm:PinHeader_1x02_P2.54mm_Vertical
- removed J6: Conn_01x04, Connector_PinHeader_2.54mm:PinHeader_1x04_P2.54mm_Vertical
- added J13: Conn_01x01, TestPoint:TestPoint_Pad_1.0x1.0mm, F.Cu at (113.8, 60.8)
- added J16: Conn_01x01, Connector_PinHeader_2.54mm:PinHeader_1x01_P2.54mm_Vertical, F.Cu at (134.8, 100.5)
- added J7: Conn_01x01, TestPoint:TestPoint_Pad_1.0x1.0mm, F.Cu at (136.8, 60.8)
- added J8: Conn_01x01, Connector_PinHeader_2.54mm:PinHeader_1x01_P2.54mm_Vertical, F.Cu at (127.2, 100.5)
- D14, D15, D16: moved to F.Cu
- J15: value Conn_01x03 -> Conn_01x01; footprint Connector_PinHeader_2.54mm:PinHeader_1x03_P2.54mm_Vertical -> Connector_PinHeader_2.54mm:PinHeader_1x01_P2.54mm_Vertical
- R21, R25: moved to B.Cu
- moved R26 85.7 mm to (104.5, 92.2), turned to -90 degrees
- moved D14 82.2 mm to (108.2, 95.2), turned to 90 degrees
- moved D13 80.7 mm to (108.2, 95.2), turned to 90 degrees
- moved D15 78.9 mm to (114.0, 95.2), turned to 90 degrees
- moved D16 76.5 mm to (119.8, 95.2), turned to 90 degrees
- moved D12 73.9 mm to (114.0, 95.2), turned to 90 degrees
- moved J15 70.6 mm to (131.0, 100.5)
- moved R25 69.3 mm to (123.2, 92.2), turned to -90 degrees
- moved D11 67.6 mm to (119.8, 95.2), turned to 90 degrees
- moved C48 33.1 mm to (147.2, 72.2), turned to 180 degrees
- moved R21 32.1 mm to (151.0, 86.0), turned to -90 degrees
- moved SW1 0.71 mm to (153.2, 76.2)
- moved D10 0.35 mm to (109.0, 78.2)
- moved D4 0.35 mm to (109.0, 76.2)
- moved R18 0.35 mm to (106.2, 76.2)
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Connections:
- J15 pad 1: VBUS_A -> +3V3_B
Routing:
- net +3V3_A: track 118.9 -> 190.0 mm, vias 10 -> 12
- net +3V3_B: track 70.5 -> 138.6 mm, vias 5 -> 8
- net GPIO7_A: track 0.00 -> 34.6 mm, vias 0 -> 1
- net GPIO23_A: track 0.00 -> 33.0 mm, vias 0 -> 2
- net GPIO20_A: track 0.00 -> 28.9 mm
- net GND: track 3.41 -> 29.9 mm, vias 0 -> 22
- net GPIO23_B: track 0.00 -> 16.3 mm, vias 0 -> 1
- net VBUS_A: track 32.6 -> 40.5 mm, vias 0 -> 1
- net Net-(D15-DOUT): track 0.00 -> 5.91 mm
- net Net-(D14-DOUT): track 0.00 -> 5.91 mm
- net Net-(D12-DOUT): track 0.00 -> 5.91 mm
- net Net-(D11-DOUT): track 0.00 -> 5.91 mm
- net VBUS_B: track 25.2 -> 28.7 mm, vias 2 -> 3
- net GPIO19_A: track 57.1 -> 59.5 mm
- net GPIO18_A: track 60.2 -> 62.4 mm
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- added copper zone on B.Cu, net GND
- added copper zone on F.Cu, net GND
Other:
- board text added: "3V3A"
- board text added: "3V3B"
- board text added: "GND"
- board text added: "J15"
- board text added: "J16"
- board text added: "J8"

Commit message: 08192026 - starting to wrap up pcb work!
Parts:
- added J17: Conn_01x01, TestPoint:TestPoint_Pad_D1.0mm, F.Cu at (128.8, 75.2)
- added J18: Conn_01x01, TestPoint:TestPoint_Pad_D1.0mm, F.Cu at (126.5, 75.2)
- added J19: Conn_01x01, TestPoint:TestPoint_Pad_D1.0mm, F.Cu at (124.2, 75.2)
- added J22: Conn_01x01, TestPoint:TestPoint_Pad_D1.0mm, F.Cu at (110.0, 86.0)
- added J6: Conn_01x01, TestPoint:TestPoint_Pad_D1.0mm, F.Cu at (131.0, 75.2)
- added J9: Conn_01x01, TestPoint:TestPoint_Pad_D1.0mm, F.Cu at (107.2, 86.0)
- moved R25 1.77 mm to (122.0, 91.0), turned to 180 degrees
- moved C46 0.25 mm to (132.7, 64.8)
- moved C18 0.22 mm to (106.0, 61.0)
- moved R8 0.15 mm to (108.1, 60.8)
- moved C2 0.10 mm to (148.7, 77.8)
Routing:
- net GND: track 29.9 -> 245.6 mm, vias 22 -> 89
- net GPIO2_A: track 27.3 -> 32.7 mm
- net GPIO1_A: track 27.7 -> 33.1 mm
- net GPIO16_A: track 37.1 -> 41.7 mm, vias 2 -> 3
- net GPIO0_B: track 29.2 -> 32.2 mm
- net Net-(D14-DIN): track 0.00 -> 2.12 mm
- net GPIO16_B: track 37.0 -> 38.9 mm
- net GPIO0_A: track 29.5 -> 31.3 mm
- net GPIO23_B: track 16.3 -> 17.2 mm
- net GPIO6_A: track 44.5 -> 45.2 mm
- net Net-(U7-OUTL): track 8.11 -> 7.53 mm
- net GPIO10_B: track 29.0 -> 28.5 mm
- net +3V3_B: track 138.6 -> 138.9 mm, vias 8 -> 10
Other:
- board text added: "0A 3B"
- board text added: "16A 17B"
- board text added: "17A 16B"
- board text added: "1A 1B"
- board text added: "2A 2B"
- board text added: "3A 0B"
- board text added: "A"
- board text added: "B"

Commit message: 08212026 - catch up and tons of silkscreen art and fun!
Parts:
- added G***: LOGO, LOGO, F.Cu at (146.8, 61.5)
- added G***: LOGO, LOGO, F.Cu at (109.0, 61.0)
- added G***: LOGO, LOGO, F.Cu at (131.0, 61.0)
- added G***: LOGO, LOGO, F.Cu at (128.0, 45.0)
- added G***: LOGO, LOGO, F.Cu at (139.5, 52.5)
- added G***: LOGO, LOGO, B.Cu at (108.8, 89.0)
- added G***: LOGO, LOGO, B.Cu at (150.4, 52.5)
- added G***: LOGO, LOGO, B.Cu at (127.3, 137.2)
- added G***: LOGO, LOGO, B.Cu at (146.8, 61.5)
- added J20: Conn_01x01, TestPoint:TestPoint_Pad_D1.0mm, B.Cu at (139.5, 90.5)
- added J21: Conn_01x01, TestPoint:TestPoint_Pad_D1.0mm, B.Cu at (108.8, 86.0)
- C48, D5, R24: moved to B.Cu
- moved J18 5.71 mm to (131.8, 73.0)
- moved J19 5.71 mm to (129.5, 73.0)
- moved C48 2.83 mm to (149.2, 70.2), turned to 90 degrees
- moved J22 1.25 mm to (108.8, 86.0)
- moved J9 1.25 mm to (106.0, 86.0)
- moved J17 0.75 mm to (129.5, 75.2)
- moved J6 0.75 mm to (131.8, 75.2)
- moved D5 0.25 mm to (151.8, 104.2)
- moved R24 0.25 mm to (154.5, 104.2)
Routing:
- net RUN_A: track 0.00 -> 12.5 mm, vias 0 -> 2
- net GND: track 245.6 -> 256.4 mm, vias 89 -> 114
- net RUN_B: track 0.00 -> 10.4 mm, vias 0 -> 2
- net GPIO2_A: track 32.7 -> 38.5 mm
- net GPIO0_B: track 32.2 -> 37.0 mm
- net +3V3_A: track 189.5 -> 193.4 mm, vias 12 -> 14
- net GPIO16_B: track 38.9 -> 40.1 mm
- net GPIO16_A: track 41.7 -> 43.0 mm
- net GPIO1_A: track 33.1 -> 33.8 mm
- net GPIO23_B: track 17.2 -> 18.0 mm
- net GPIO10_A: track 26.1 -> 26.0 mm, vias 1 -> 2
Other:
- board text added: "...one for each tool head?"
- board text added: "HenryLi-0/river"
- board text added: "MCU A"
- board text added: "MCU B"
- board text added: "Ozone"
- board text added: "POWER"
- board text added: "RUN_A"
- board text added: "RUN_B"
- board text added: "by henryli-0"
- board text added: "lazors!!1"
- board text added: "o"
- board text added: "{dblquote}Only those that risk going too far can possibly know how far they can go.{dblquote} - Walter Bishop, Fringe"

Commit message: more silkscreen art! and back to wrapping up
Parts:
- added G***: LOGO, LOGO, B.Cu at (161.0, 95.5)
- moved D5 3.01 mm to (154.8, 104.5), turned to 90 degrees
- moved R24 3.01 mm to (154.8, 107.2), turned to -90 degrees
Routing:
- net GPIO10_A: track 26.0 -> 29.6 mm

Commit message: 08232026 - exporting and back to again
Other:
- board text added: "Graciously Funded By Hack Club!!!"
- board text added: "v1.0"
Changed lines of the file:
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@@
 	)
 	(paper "A4")
+	(title_block
+		(title "River Board PCB")
+		(date "2026-08-23")
+		(rev "1.0")
+	)
 	(layers
 		(0 "F.Cu" signal)
@@
 			(plot_on_all_layers_selection 0x0000000_00000000)
 			(disableapertmacros no)
-			(usegerberextensions no)
+			(usegerberextensions yes)
 			(usegerberattributes yes)
 			(usegerberadvancedattributes yes)
-			(creategerberjobfile yes)
+			(creategerberjobfile no)
 			(dashed_line_dash_ratio 12.000000)
 			(dashed_line_gap_ratio 3.000000)
@@
 			(psa4output no)
 			(plotreference yes)
-			(plotvalue yes)
+			(plotvalue no)
 			(plotfptext yes)
 			(plotinvisibletext no)
 			(sketchpadsonfab no)
-			(subtractmaskfromsilk no)
+			(subtractmaskfromsilk yes)
 			(outputformat 1)
 			(mirror no)
-			(drillshape 1)
+			(drillshape 0)
 			(scaleselection 1)
-			(outputdirectory "")
+			(outputdirectory "production/")
 		)
 	)
@@
 			(at -0.55 -0.55 270)
 			(size 0.5 0.5)
-			(drill 0.3)
+			(drill 0.2)
 			(property pad_prop_heatsink)
 			(layers "*.Cu")
@@
 			(at -0.55 0.55 270)
 			(size 0.5 0.5)
-			(drill 0.3)
+			(drill 0.2)
 			(property pad_prop_heatsink)
 			(layers "*.Cu")
@@
 			(at 0.55 -0.55 270)
 			(size 0.5 0.5)
-			(drill 0.3)
+			(drill 0.2)
 			(property pad_prop_heatsink)
 			(layers "*.Cu")
@@
 			(at 0.55 0.55 270)
 			(size 0.5 0.5)
-			(drill 0.3)
+			(drill 0.2)
 			(property pad_prop_heatsink)
 			(layers "*.Cu")
@@
 		)
 	)
+	(gr_text "v1.0"
+		(at 151.5 54.75 0)
+		(layer "F.SilkS")
+		(effects
+			(font
+				(size 0.8 0.8)
+				(thickness 0.2)
+				(bold yes)
+			)
+		)
+	)
 	(gr_text "GND"
 		(at 134.75 103 0)
@@
 		)
 	)
+	(gr_text "Graciously Funded By Hack Club!!!"
+		(at 121.25 64.75 0)
+		(layer "F.SilkS")
+		(effects
+			(font
+				(size 0.8 0.8)
+				(thickness 0.2)
+				(bold yes)
+			)
+		)
+	)
 	(gr_text "2A\n2B"
 		(at 133.5 73 0)
@@
 	)
 	(gr_text "...one for each tool head?"
-		(at 101.25 115.75 -90)
+		(at 101.25 115.75 90)
 		(layer "F.SilkS")
 		(effects
