File: pcb/board/board.kicad_pcb (KiCad board)
At the start: 2 copper layers, 56 x 80 mm, 138 parts, among them J1 (A) USB_C_Receptacle_USB2.0_1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, J10 OLED_128x32, J11 LCD_128x160, J12 AudioJack3, J13 Conn_01x01, J14 Micro_SD_Card, J15 Conn_01x01, J16 Conn_01x01, J17 Conn_01x01, J18 Conn_01x01, J19 Conn_01x01, J2 (B) USB_C_Receptacle_USB2.0_1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, J20 Conn_01x01, J21 Conn_01x01, J22 Conn_01x01, J3 (C) USB_C_Receptacle_USB2.0_1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, J6 Conn_01x01, J7 Conn_01x01, J8 Conn_01x01, J9 Conn_01x01, SW1 SW_Push, SW2 SW_Push, SW3 Switch, SW4 Switch, SW5 Switch, SW6 RotaryEncoder_Switch, U1 RP2040, U2 NCP1117-3.3_SOT223, U3 W25Q16JVZPIQ TR, U4 NCP1117-3.3_SOT223, U5 RP2040, U6 W25Q16JVZPIQ TR, U7 PCM5101A, U8 TLV70033_SOT23-5, U9 TPA6132A2RTE, Y1 12MHz, Y2 12MHz

Commit message: update micro sd card footprint
Parts:
- J14: footprint Connector_Card:microSD_HC_Wuerth_693072010801 -> Connector_Card:microSD_HC_Molex_47219-2001
- moved J14 0.50 mm to (144.2, 105.2)
- moved C48 0.25 mm to (138.5, 96.8)
Routing:
- net GND: track 383.3 -> 386.1 mm, vias 152 -> 170
- net GPIO19_A: track 59.2 -> 58.7 mm
Other:
- board text added: "v1.0 r1"
- board text removed: "v1.0"
